File: ember-pcb.kicad_pcb (KiCad board)
At the start: 6 copper layers, 119.3 x 94.2 mm, 35 parts, among them J1 Samtec_ASP-134486-01, J2 Conn_Coaxial_Power, J3 Conn_02x12_Odd_Even, J4 Conn_01x07, J5 Conn_Coaxial_Power, SW1 SW_SP3T, SW2 SW_SP3T, SW3 SW_DIP_x02, U1 EMBER Macro, U2 LP5912-0.9DRV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

Commit message: 6 layer
Parts:
- removed J1: Samtec_ASP-134486-01, Connector_Samtec:Samtec_FMC_ASP-134486-01_10x40_P1.27mm_Vertical
Routing:
- net /vddio: track 230.9 -> 108.6 mm, vias 2 -> 0
- net /vddio_fsm: track 231.5 -> 117.6 mm, vias 1 -> 0
- net /vdd_fsm: track 214.9 -> 120.7 mm
- net /wl_source_pin: track 55.2 -> 121.0 mm
- net /vdd_test: track 90.4 -> 129.1 mm
- net /vddio_dac: track 222.6 -> 248.4 mm, vias 1 -> 4
- net /vdd: track 185.3 -> 159.9 mm
- net /vdd_dac: track 200.2 -> 176.4 mm
- net GND: track 404.0 -> 383.0 mm
- net /iref_test: track 131.8 -> 137.8 mm
- net /vsa: track 218.2 -> 213.8 mm, vias 0 -> 4
- net /byp: track 90.9 -> 88.2 mm
- net /sl_source_pin: track 65.0 -> 66.6 mm
- net /man: track 81.3 -> 79.8 mm
- net /bl_source_pin: track 75.1 -> 74.2 mm
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- added copper zone on F.Cu, net /vdd
- added copper zone on In2.Cu, net /vdd
- added copper zone on F.Cu, net /vdd_dac
- added copper zone on In2.Cu, net /vdd_dac
- added copper zone on F.Cu, net /vdd_fsm
- added copper zone on In2.Cu, net /vdd_fsm
- added copper zone on In2.Cu, net /vddio
- added copper zone on In2.Cu, net /vddio_dac
- added copper zone on F.Cu, net /vddio_fsm
- added copper zone on In2.Cu, net /vddio_fsm
- removed copper zone on In1.Cu, net /vddio_fsm
