File: ember-pcb.kicad_sch (KiCad schematic)
At the start: 35 parts, among them J1 Samtec_ASP-134486-01, J2 Conn_Coaxial_Power, J3 Conn_02x12_Odd_Even, J4 Conn_01x07, J5 Conn_Coaxial_Power, SW1 SW_SP3T, SW2 SW_SP3T, SW3 SW_DIP_x02, U1 EMBER Macro, U2 LP5912-0.9DRV, U3 LP5912-1.1DRV, U4 LP5912-2.5DRV

Commit message: Getting more in shape
Parts:
- C1, C3, C6, C8: footprint Capacitor_SMD:CP_Elec_3x5.3 -> Capacitor_Tantalum_SMD:CP_EIA-3528-21_Kemet-B
- C10, C2, C5, C7: footprint Capacitor_SMD:CP_Elec_3x5.3 -> Capacitor_SMD:C_1210_3225Metric
- C4, C9: footprint Capacitor_SMD:CP_Elec_3x5.3 -> Capacitor_Tantalum_SMD:CP_EIA-3528-12_Kemet-T
- J1: value Samtec_ASP-134486-01 -> Samtec_ASP-134602-01; footprint Connector_Samtec:Samtec_FMC_ASP-134486-01_10x40_P1.27mm_Vertical -> Connector_Samtec:Samtec_FMC_ASP-134602-01_10x40_P1.27mm_Vertical; symbol Connector:Samtec_ASP-134486-01 -> Connector:Samtec_ASP-134602-01
- J2, J5: footprint Connector_Coaxial:SMA_Samtec_SMA-J-P-X-ST-EM1_EdgeMount -> Connector_Coaxial:SMA_Molex_73251-2200_Horizontal
- U1: footprint ember-pcb:ZIF-441_Aries -> ZIF:ARIES_441-PRS21001-12
Connections:
- net GND: now also U1.U18 (vss), U1.U3 (vss), U1.V7 (vss), U1.W1 (vss), U1.W15 (vss), U1.W20 (vss); no longer U1.V18 (vss), U1.V3 (vss), U1.W7 (vss), U1.Y1 (vss), U1.Y15 (vss), U1.Y20 (vss)
- net aclk: now also U1.U7 (aclk); no longer J1.K38 (Pin_38), U1.V7 (aclk)
- net bl_en: now also U1.S2 (bl_en); no longer J1.C14 (Pin_14), U1.T2 (bl_en)
- net bl_source_pin: now also U1.W3 (bl_source_pin); no longer U1.Y3 (bl_source_pin)
- net bleed_en: no longer J1.G22 (Pin_22)
- net bsl_dac_config_0: now also U1.T7 (bsl_dac_config_0); no longer J1.K11 (Pin_11), U1.U7 (bsl_dac_config_0)
- net bsl_dac_config_1: now also U1.U6 (bsl_dac_config_1); no longer J1.J9 (Pin_9), U1.V6 (bsl_dac_config_1)
- net bsl_dac_config_2: now also U1.T6 (bsl_dac_config_2); no longer J1.H11 (Pin_11), U1.U6 (bsl_dac_config_2)
- net bsl_dac_config_3: now also U1.U5 (bsl_dac_config_3); no longer J1.G9 (Pin_9), U1.V5 (bsl_dac_config_3)
- net bsl_dac_config_4: now also U1.T5 (bsl_dac_config_4); no longer J1.F11 (Pin_11), U1.U5 (bsl_dac_config_4)
- net bsl_dac_en: now also U1.T4 (bsl_dac_en); no longer J1.D11 (Pin_11), U1.U4 (bsl_dac_en)
- net byp: now also U1.W8 (byp); no longer U1.Y8 (byp)
- net clamp_ref_0: now also U1.V2 (clamp_ref_0); no longer J1.E7 (Pin_7), U1.W2 (clamp_ref_0)
- net clamp_ref_1: now also U1.S4 (clamp_ref_1); no longer J1.F14 (Pin_14), U1.T4 (clamp_ref_1)
- net clamp_ref_2: now also U1.T3 (clamp_ref_2); no longer J1.C10 (Pin_10), U1.U3 (clamp_ref_2)
- net clamp_ref_3: no longer J1.E15 (Pin_15)
- net clamp_ref_4: now also U1.S3 (clamp_ref_4); no longer J1.D14 (Pin_14), U1.T3 (clamp_ref_4)
- net clamp_ref_5: no longer J1.G16 (Pin_16)
- net di_0: no longer J1.F16 (Pin_16)
- net di_1: now also U1.S1 (di_1); no longer J1.K13 (Pin_13), U1.T1 (di_1)
- net di_10: no longer J1.H19 (Pin_19)
- net di_11: no longer J1.F19 (Pin_19)
- net di_12: no longer J1.F20 (Pin_20)
- net di_13: no longer J1.K20 (Pin_20)
- net di_14: no longer J1.J21 (Pin_21)
- net di_15: no longer J1.H20 (Pin_20)
- net di_16: no longer J1.C23 (Pin_23)
- net di_17: no longer J1.C22 (Pin_22)
- net di_18: no longer J1.E24 (Pin_24)
- net di_19: no longer J1.F22 (Pin_22)
- net di_2: no longer J1.H17 (Pin_17)
- net di_20: no longer J1.E22 (Pin_22)
- net di_21: no longer J1.D23 (Pin_23)
- net di_22: no longer J1.F23 (Pin_23)
- net di_23: no longer J1.F26 (Pin_26)
- net di_24: no longer J1.G24 (Pin_24)
- net di_25: no longer J1.G25 (Pin_25)
- net di_26: no longer J1.J24 (Pin_24)
- net di_27: no longer J1.J27 (Pin_27)
- net di_28: no longer J1.H25 (Pin_25)
- net di_29: no longer J1.J25 (Pin_25)
- net di_3: no longer J1.D15 (Pin_15)
- net di_30: no longer J1.H26 (Pin_26)
- net di_31: no longer J1.K26 (Pin_26)
- net di_32: no longer J1.E28 (Pin_28)
- net di_33: no longer J1.F28 (Pin_28)
- net di_34: no longer J1.F35 (Pin_35)
- net di_35: no longer J1.G28 (Pin_28)
- net di_36: no longer J1.G37 (Pin_37)
- net di_37: no longer J1.J31 (Pin_31)
- net di_38: no longer J1.H28 (Pin_28)
- net di_39: no longer J1.K31 (Pin_31)
- net di_4: no longer J1.F17 (Pin_17)
- net di_40: no longer J1.J28 (Pin_28)
- net di_41: no longer J1.F32 (Pin_32)
- net di_42: no longer J1.H32 (Pin_32)
- net di_43: no longer J1.K28 (Pin_28)
- net di_44: no longer J1.K32 (Pin_32)
- net di_45: no longer J1.E33 (Pin_33)
- net di_46: no longer J1.F29 (Pin_29)
- net di_47: no longer J1.H37 (Pin_37)
- net di_5: no longer J1.E18 (Pin_18)
- net di_6: no longer J1.G18 (Pin_18)
- net di_7: no longer J1.D18 (Pin_18)
- net di_8: no longer J1.D17 (Pin_17)
- net di_9: no longer J1.G19 (Pin_19)
- net heartbeat: now also U1.T10 (heartbeat); no longer U1.U10 (heartbeat)
- net man: now also U1.U10 (man); no longer U1.V10 (man)
- net mclk_pause: now also U1.T8 (mclk_pause); no longer J1.G7 (Pin_7), U1.U8 (mclk_pause)
- net miso: now also U1.V9 (miso); no longer J1.H7 (Pin_7), U1.W9 (miso)
- net mosi: now also U1.T9 (mosi); no longer J1.H8 (Pin_8), U1.U9 (mosi)
- net read_dac_config_0: no longer J1.F37 (Pin_37)
- net read_dac_config_1: no longer J1.C27 (Pin_27)
- net read_dac_config_2: no longer J1.H31 (Pin_31)
- net read_dac_config_3: no longer J1.K25 (Pin_25)
- net read_dac_en: now also U1.U4 (read_dac_en); no longer J1.E9 (Pin_9), U1.V4 (read_dac_en)
- net read_ref_0: no longer J1.H29 (Pin_29)
- net read_ref_1: no longer J1.K35 (Pin_35)
- net read_ref_2: no longer J1.E36 (Pin_36)
- net read_ref_3: no longer J1.K29 (Pin_29)
- net read_ref_4: no longer J1.J37 (Pin_37)
- net read_ref_5: no longer J1.J33 (Pin_33)
- net rram_addr_0: no longer J1.K37 (Pin_37)
- net rram_addr_1: no longer J1.G36 (Pin_36)
- net rram_addr_10: no longer J1.H38 (Pin_38)
- net rram_addr_11: no longer J1.H34 (Pin_34)
- net rram_addr_12: no longer J1.E31 (Pin_31)
- net rram_addr_13: no longer J1.J34 (Pin_34)
- net rram_addr_14: no longer J1.F31 (Pin_31)
- net rram_addr_15: no longer J1.K34 (Pin_34)
- net rram_addr_2: no longer J1.F38 (Pin_38)
- net rram_addr_3: no longer J1.E30 (Pin_30)
- net rram_addr_4: no longer J1.E34 (Pin_34)
- net rram_addr_5: no longer J1.F34 (Pin_34)
- net rram_addr_6: no longer J1.J36 (Pin_36)
- net rram_addr_7: no longer J1.G30 (Pin_30)
- net rram_addr_8: no longer J1.G34 (Pin_34)
- net rram_addr_9: no longer J1.J30 (Pin_30)
- net rst_n: no longer J1.D9 (Pin_9)
- net sa_clk: now also U1.W7 (sa_clk); no longer J1.E2 (Pin_2), U1.Y7 (sa_clk)
- net sa_do_0: no longer J1.J22 (Pin_22)
- net sa_do_1: no longer J1.E21 (Pin_21)
- net sa_do_10: no longer J1.K16 (Pin_16)
- net sa_do_11: no longer J1.J18 (Pin_18)
- net sa_do_12: no longer J1.C19 (Pin_19)
- net sa_do_13: no longer J1.C18 (Pin_18)
- net sa_do_14: no longer J1.K17 (Pin_17)
- net sa_do_15: now also U1.S20 (sa_do_15); no longer J1.C15 (Pin_15), U1.T20 (sa_do_15)
- net sa_do_16: no longer J1.J16 (Pin_16)
- net sa_do_17: no longer J1.E16 (Pin_16)
- net sa_do_18: no longer J1.H16 (Pin_16)
- net sa_do_19: now also U1.T20 (sa_do_19); no longer J1.J13 (Pin_13), U1.U20 (sa_do_19)
- net sa_do_2: no longer J1.D24 (Pin_24)
- net sa_do_20: no longer J1.J15 (Pin_15)
- net sa_do_21: no longer J1.G15 (Pin_15)
- net sa_do_22: now also U1.S18 (sa_do_22); no longer J1.K14 (Pin_14), U1.T18 (sa_do_22)
- net sa_do_23: now also U1.S17 (sa_do_23); no longer J1.H14 (Pin_14), U1.T17 (sa_do_23)
- net sa_do_24: now also U1.T18 (sa_do_24); no longer J1.H13 (Pin_13), U1.U18 (sa_do_24)
- net sa_do_25: now also U1.T17 (sa_do_25); no longer J1.G13 (Pin_13), U1.U17 (sa_do_25)
- net sa_do_26: now also U1.V19 (sa_do_26); no longer J1.K8 (Pin_8), U1.W19 (sa_do_26)
- net sa_do_27: now also U1.T16 (sa_do_27); no longer J1.F13 (Pin_13), U1.U16 (sa_do_27)
- net sa_do_28: now also U1.U17 (sa_do_28); no longer J1.K10 (Pin_10), U1.V17 (sa_do_28)
- net sa_do_29: now also U1.T15 (sa_do_29); no longer J1.E13 (Pin_13), U1.U15 (sa_do_29)
- net sa_do_3: no longer J1.D21 (Pin_21)
- net sa_do_30: now also U1.U16 (sa_do_30); no longer J1.J10 (Pin_10), U1.V16 (sa_do_30)
- net sa_do_31: now also U1.V17 (sa_do_31); no longer J1.F8 (Pin_8), U1.W17 (sa_do_31)
- net sa_do_32: now also U1.T14 (sa_do_32); no longer J1.J12 (Pin_12), U1.U14 (sa_do_32)
- net sa_do_33: now also U1.U15 (sa_do_33); no longer J1.H10 (Pin_10), U1.V15 (sa_do_33)
- net sa_do_34: now also U1.U14 (sa_do_34); no longer J1.G10 (Pin_10), U1.V14 (sa_do_34)
- net sa_do_35: now also U1.W16 (sa_do_35); no longer J1.J6 (Pin_6), U1.Y16 (sa_do_35)
- net sa_do_36: now also U1.T13 (sa_do_36); no longer J1.G12 (Pin_12), U1.U13 (sa_do_36)
- net sa_do_37: now also U1.U13 (sa_do_37); no longer J1.F10 (Pin_10), U1.V13 (sa_do_37)
- net sa_do_38: now also U1.U12 (sa_do_38); no longer J1.E10 (Pin_10), U1.V12 (sa_do_38)
- net sa_do_39: now also U1.T12 (sa_do_39); no longer J1.E12 (Pin_12), U1.U12 (sa_do_39)
- net sa_do_4: no longer J1.K22 (Pin_22)
- net sa_do_40: now also U1.W14 (sa_do_40); no longer J1.E6 (Pin_6), U1.Y14 (sa_do_40)
- net sa_do_41: now also U1.V12 (sa_do_41); no longer J1.J7 (Pin_7), U1.W12 (sa_do_41)
- net sa_do_42: now also U1.V13 (sa_do_42); no longer J1.K7 (Pin_7), U1.W13 (sa_do_42)
- net sa_do_43: now also U1.U11 (sa_do_43); no longer J1.C11 (Pin_11), U1.V11 (sa_do_43)
- net sa_do_44: now also U1.W13 (sa_do_44); no longer J1.F5 (Pin_5), U1.Y13 (sa_do_44)
- net sa_do_45: now also U1.T11 (sa_do_45); no longer J1.D12 (Pin_12), U1.U11 (sa_do_45)
- net sa_do_46: now also U1.W12 (sa_do_46); no longer J1.F4 (Pin_4), U1.Y12 (sa_do_46)
- net sa_do_47: now also U1.V11 (sa_do_47); no longer J1.F7 (Pin_7), U1.W11 (sa_do_47)
- net sa_do_5: no longer J1.G21 (Pin_21)
- net sa_do_6: no longer J1.D20 (Pin_20)
- net sa_do_7: no longer J1.J19 (Pin_19)
- net sa_do_8: no longer J1.K19 (Pin_19)
- net sa_do_9: no longer J1.E19 (Pin_19)
- net sa_en: no longer J1.H35 (Pin_35)
- net sa_rdy: now also U1.V10 (sa_rdy); no longer J1.E3 (Pin_3), U1.W10 (sa_rdy)
- net sc: now also U1.U9 (sc); no longer J1.D8 (Pin_8), U1.V9 (sc)
- net sclk: now also U1.U8 (sclk); no longer J1.G6 (Pin_6), U1.V8 (sclk)
- net set_rst: no longer J1.G33 (Pin_33)
- net sl_en: no longer J1.E37 (Pin_37)
- net sl_source_pin: now also U1.V6 (sl_source_pin); no longer U1.W6 (sl_source_pin)
- net vdd: now also U1.T19 (vdd), U1.U1 (vdd), U1.V14 (vdd), U1.W6 (vdd); no longer U1.U19 (vdd), U1.V1 (vdd), U1.W14 (vdd), U1.Y6 (vdd)
- net vdd_dac: now also U1.U19 (vdd_dac), U1.V1 (vdd_dac), U1.W9 (vdd_dac); no longer U1.V19 (vdd_dac), U1.W1 (vdd_dac), U1.Y9 (vdd_dac)
- net vdd_fsm: now also U1.V5 (vdd_fsm), U1.W17 (vdd_fsm); no longer U1.W5 (vdd_fsm), U1.Y17 (vdd_fsm)
- net vddio: now also U1.U2 (vddio), U1.V20 (vddio), U1.V3 (vddio), U1.W11 (vddio), U1.W19 (vddio); no longer U1.V2 (vddio), U1.W20 (vddio), U1.W3 (vddio), U1.Y11 (vddio), U1.Y19 (vddio)
- net vddio_dac: now also U1.S19 (vddio_dac), U1.T1 (vddio_dac), U1.V16 (vddio_dac), U1.W10 (vddio_dac), U1.W4 (vddio_dac); no longer U1.T19 (vddio_dac), U1.U1 (vddio_dac), U1.W16 (vddio_dac), U1.Y10 (vddio_dac), U1.Y4 (vddio_dac)
- net vddio_fsm: now also U1.T2 (vddio_fsm), U1.U20 (vddio_fsm), U1.V15 (vddio_fsm), U1.V18 (vddio_fsm), U1.V8 (poc), U1.W2 (vddio_fsm), U1.W5 (vddio_fsm); no longer U1.U2 (vddio_fsm), U1.V20 (vddio_fsm), U1.W15 (vddio_fsm), U1.W18 (vddio_fsm), U1.W8 (poc), U1.Y2 (vddio_fsm), U1.Y5 (vddio_fsm)
- net vsa: now also U1.V4 (vsa), U1.W18 (vsa); no longer U1.W4 (vsa), U1.Y18 (vsa)
- net we: no longer J1.G31 (Pin_31)
- net wl_dac_config_0: no longer J1.D27 (Pin_27)
- net wl_dac_config_1: no longer J1.E25 (Pin_25)
- net wl_dac_config_2: no longer J1.C26 (Pin_26)
- net wl_dac_config_3: no longer J1.E27 (Pin_27)
- net wl_dac_config_4: no longer J1.F25 (Pin_25)
- net wl_dac_config_5: no longer J1.G27 (Pin_27)
- net wl_dac_config_6: no longer J1.H23 (Pin_23)
- net wl_dac_config_7: no longer J1.D26 (Pin_26)
- net wl_dac_en: no longer J1.K23 (Pin_23)
- net wl_en: no longer J1.H22 (Pin_22)

Commit message: Commit
Parts:
- added H4: MountingHole, MountingHole:MountingHole_2.5mm, symbol Mechanical:MountingHole
- added J3: Conn_02x40_Top_Bottom, Connector_PinHeader_1.27mm:PinHeader_2x40_P1.27mm_Vertical, symbol Connector_Generic:Conn_02x40_Top_Bottom
- renumbered J3 to J4, J4 to J5, J5 to J6
Connections:
- net pin_30: now reaches J1.D11 (Pin_11)
- net pin_34: now reaches J1.D12 (Pin_12)
- net pin_45: now reaches J1.D14 (Pin_14)
- net pin_50: now reaches J1.D15 (Pin_15)
- net pin_60: now reaches J1.D17 (Pin_17)
- net pin_65: now reaches J1.D18 (Pin_18)
- net pin_76: now reaches J1.D20 (Pin_20)
- net pin_80: now reaches J1.D21 (Pin_21)
- net pin_92: now reaches J1.D23 (Pin_23)
- net pin_96: now reaches J1.D24 (Pin_24)
- net pin_107: now reaches J1.D26 (Pin_26)
- net pin_112: now reaches J1.D27 (Pin_27)
- net at J1.D30 (Pin_30): now also J1.D31 (Pin_31)
- net pin_14: now reaches J1.D8 (Pin_8)
- net pin_18: now reaches J1.D9 (Pin_9)
- net pin_24: now reaches J1.F10 (Pin_10)
- net pin_31: now reaches J1.F11 (Pin_11)
- net pin_39: now reaches J1.F13 (Pin_13)
- net pin_46: now reaches J1.F14 (Pin_14)
- net pin_55: now reaches J1.F16 (Pin_16)
- net pin_61: now reaches J1.F17 (Pin_17)
- net pin_71: now reaches J1.F19 (Pin_19)
- net pin_77: now reaches J1.F20 (Pin_20)
- net pin_86: now reaches J1.F22 (Pin_22)
- net pin_93: now reaches J1.F23 (Pin_23)
- net pin_101: now reaches J1.F25 (Pin_25)
- net pin_108: now reaches J1.F26 (Pin_26)
- net pin_117: now reaches J1.F28 (Pin_28)
- net pin_122: now reaches J1.F29 (Pin_29)
- net pin_129: now reaches J1.F31 (Pin_31)
- net pin_134: now reaches J1.F32 (Pin_32)
- net pin_141: now reaches J1.F34 (Pin_34)
- net pin_146: now reaches J1.F35 (Pin_35)
- net pin_153: now reaches J1.F37 (Pin_37)
- net pin_158: now reaches J1.F38 (Pin_38)
- net pin_3: now reaches J1.F4 (Pin_4)
- net pin_4: now reaches J1.F5 (Pin_5)
- net pin_9: now reaches J1.F7 (Pin_7)
- net pin_15: now reaches J1.F8 (Pin_8)
- net pin_22: now reaches J1.C10 (Pin_10)
- net pin_29: now reaches J1.C11 (Pin_11)
- net pin_44: now reaches J1.C14 (Pin_14)
- net pin_49: now reaches J1.C15 (Pin_15)
- net pin_64: now reaches J1.C18 (Pin_18)
- net pin_69: now reaches J1.C19 (Pin_19)
- net pin_84: now reaches J1.C22 (Pin_22)
- net pin_91: now reaches J1.C23 (Pin_23)
- net pin_106: now reaches J1.C26 (Pin_26)
- net pin_111: now reaches J1.C27 (Pin_27)
- net pin_26: now reaches J1.H10 (Pin_10)
- net pin_32: now reaches J1.H11 (Pin_11)
- net pin_41: now reaches J1.H13 (Pin_13)
- net pin_47: now reaches J1.H14 (Pin_14)
- net pin_57: now reaches J1.H16 (Pin_16)
- net pin_62: now reaches J1.H17 (Pin_17)
- net pin_73: now reaches J1.H19 (Pin_19)
- net pin_78: now reaches J1.H20 (Pin_20)
- net pin_88: now reaches J1.H22 (Pin_22)
- net pin_94: now reaches J1.H23 (Pin_23)
- net pin_103: now reaches J1.H25 (Pin_25)
- net pin_109: now reaches J1.H26 (Pin_26)
- net pin_119: now reaches J1.H28 (Pin_28)
- net pin_123: now reaches J1.H29 (Pin_29)
- net pin_131: now reaches J1.H31 (Pin_31)
- net pin_135: now reaches J1.H32 (Pin_32)
- net pin_143: now reaches J1.H34 (Pin_34)
- net pin_147: now reaches J1.H35 (Pin_35)
- net pin_155: now reaches J1.H37 (Pin_37)
- net pin_159: now reaches J1.H38 (Pin_38)
- net pin_11: now reaches J1.H7 (Pin_7)
- net pin_16: now reaches J1.H8 (Pin_8)
- net pin_23: now reaches J1.E10 (Pin_10)
- net pin_35: now reaches J1.E12 (Pin_12)
- net pin_38: now reaches J1.E13 (Pin_13)
- net pin_51: now reaches J1.E15 (Pin_15)
- net pin_54: now reaches J1.E16 (Pin_16)
- net pin_66: now reaches J1.E18 (Pin_18)
- net pin_70: now reaches J1.E19 (Pin_19)
- net pin_1: now reaches J1.E2 (Pin_2)
- net pin_81: now reaches J1.E21 (Pin_21)
- net pin_85: now reaches J1.E22 (Pin_22)
- net pin_97: now reaches J1.E24 (Pin_24)
- net pin_100: now reaches J1.E25 (Pin_25)
- net pin_113: now reaches J1.E27 (Pin_27)
- net pin_116: now reaches J1.E28 (Pin_28)
- net pin_2: now reaches J1.E3 (Pin_3)
- net pin_125: now reaches J1.E30 (Pin_30)
- net pin_128: now reaches J1.E31 (Pin_31)
- net pin_137: now reaches J1.E33 (Pin_33)
- net pin_140: now reaches J1.E34 (Pin_34)
- net pin_149: now reaches J1.E36 (Pin_36)
- net pin_152: now reaches J1.E37 (Pin_37)
- net pin_5: now reaches J1.E6 (Pin_6)
- net pin_8: now reaches J1.E7 (Pin_7)
- net pin_19: now reaches J1.E9 (Pin_9)
- net pin_28: now reaches J1.K10 (Pin_10)
- net pin_33: now reaches J1.K11 (Pin_11)
- net pin_43: now reaches J1.K13 (Pin_13)
- net pin_48: now reaches J1.K14 (Pin_14)
- net pin_59: now reaches J1.K16 (Pin_16)
- net pin_63: now reaches J1.K17 (Pin_17)
- net pin_75: now reaches J1.K19 (Pin_19)
- net pin_79: now reaches J1.K20 (Pin_20)
- net pin_90: now reaches J1.K22 (Pin_22)
- net pin_95: now reaches J1.K23 (Pin_23)
- net pin_105: now reaches J1.K25 (Pin_25)
- net pin_110: now reaches J1.K26 (Pin_26)
- net pin_121: now reaches J1.K28 (Pin_28)
- net pin_124: now reaches J1.K29 (Pin_29)
- net pin_133: now reaches J1.K31 (Pin_31)
- net pin_136: now reaches J1.K32 (Pin_32)
- net pin_145: now reaches J1.K34 (Pin_34)
- net pin_148: now reaches J1.K35 (Pin_35)
- net pin_157: now reaches J1.K37 (Pin_37)
- net pin_160: now reaches J1.K38 (Pin_38)
- net pin_13: now reaches J1.K7 (Pin_7)
- net pin_17: now reaches J1.K8 (Pin_8)
- net pin_25: now reaches J1.G10 (Pin_10)
- net pin_36: now reaches J1.G12 (Pin_12)
- net pin_40: now reaches J1.G13 (Pin_13)
- net pin_52: now reaches J1.G15 (Pin_15)
- net pin_56: now reaches J1.G16 (Pin_16)
- net pin_67: now reaches J1.G18 (Pin_18)
- net pin_72: now reaches J1.G19 (Pin_19)
- net pin_82: now reaches J1.G21 (Pin_21)
- net pin_87: now reaches J1.G22 (Pin_22)
- net pin_98: now reaches J1.G24 (Pin_24)
- net pin_102: now reaches J1.G25 (Pin_25)
- net pin_114: now reaches J1.G27 (Pin_27)
- net pin_118: now reaches J1.G28 (Pin_28)
- net pin_126: now reaches J1.G30 (Pin_30)
- net pin_130: now reaches J1.G31 (Pin_31)
- net pin_138: now reaches J1.G33 (Pin_33)
- net pin_142: now reaches J1.G34 (Pin_34)
- net pin_150: now reaches J1.G36 (Pin_36)
- net pin_154: now reaches J1.G37 (Pin_37)
- net pin_6: now reaches J1.G6 (Pin_6)
- net pin_10: now reaches J1.G7 (Pin_7)
- net pin_20: now reaches J1.G9 (Pin_9)
- net pin_27: now reaches J1.J10 (Pin_10)
- net pin_37: now reaches J1.J12 (Pin_12)
- net pin_42: now reaches J1.J13 (Pin_13)
- net pin_53: now reaches J1.J15 (Pin_15)
- net pin_58: now reaches J1.J16 (Pin_16)
- net pin_68: now reaches J1.J18 (Pin_18)
- net pin_74: now reaches J1.J19 (Pin_19)
- net pin_83: now reaches J1.J21 (Pin_21)
- net pin_89: now reaches J1.J22 (Pin_22)
- net pin_99: now reaches J1.J24 (Pin_24)
- net pin_104: now reaches J1.J25 (Pin_25)
- net pin_115: now reaches J1.J27 (Pin_27)
- net pin_120: now reaches J1.J28 (Pin_28)
- net pin_127: now reaches J1.J30 (Pin_30)
- net pin_132: now reaches J1.J31 (Pin_31)
- net pin_139: now reaches J1.J33 (Pin_33)
- net pin_144: now reaches J1.J34 (Pin_34)
- net pin_151: now reaches J1.J36 (Pin_36)
- net pin_156: now reaches J1.J37 (Pin_37)
- net pin_7: now reaches J1.J6 (Pin_6)
- net pin_12: now reaches J1.J7 (Pin_7)
- net pin_21: now reaches J1.J9 (Pin_9)
- no-connect marks 83 -> 81
Other:
- note added: "di_36 iref_test di_47 read_ref_4 rram_addr_0 rram_addr_2 rram_addr_10 di_34 sa_en read_ref_1 read_ref_2 rram_addr_1 rram_addr_6 sl_en read_dac_config_0 di_37 di_39 di_41 di_42 di_44 di_45 set_rst read_ref_5 rram_addr_4 rram_addr_5 rram_addr_8 rram_addr_11 rram_addr_13 rram_addr_15 di_27 di_32 di_33 di_35 di_38 di_40 di_43 di_46 read_ref_0 read_ref_3 rram_addr_3 rram_addr_7 rram_addr_9 rram_addr_1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"

Commit message: Updates
Parts:
- removed J3: Conn_02x40_Top_Bottom, Connector_PinHeader_1.27mm:PinHeader_2x40_P1.27mm_Vertical, symbol Connector_Generic:Conn_02x40_Top_Bottom
- removed TP2: TestPointCorePwr, TestPoint:TestPoint_Pad_D1.0mm, symbol Connector:TestPoint
- removed TP3: TestPointGnd, TestPoint:TestPoint_Pad_D1.0mm, symbol Connector:TestPoint
- removed TP4: TestPointIOPwr, TestPoint:TestPoint_Pad_D1.0mm, symbol Connector:TestPoint
- added U5: FMC_Vias, symbol ember-lib:FMC_Vias
- renumbered J4 to J3, J5 to J4, J6 to J5
Connections:
- net GND: now also U2.7 (EP), U3.7 (EP), U4.7 (EP)
- net aclk: now also U5.216
- net bl_en: now also U5.208
- net bleed_en: now also U5.247
- net bsl_dac_config_0: now also U5.198
- net bsl_dac_config_1: now also U5.184
- net bsl_dac_config_2: now also U5.199
- net bsl_dac_config_3: now also U5.185
- net bsl_dac_config_4: now also U5.182
- net bsl_dac_en: now also U5.201
- net clamp_ref_0: now also U5.173
- net clamp_ref_1: now also U5.206
- net clamp_ref_2: now also U5.202
- net clamp_ref_3: now also U5.213
- net clamp_ref_4: now also U5.207
- net clamp_ref_5: now also U5.219
- net di_0: now also U5.220
- net di_1: now also U5.209
- net di_10: now also U5.235
- net di_11: now also U5.237
- net di_12: now also U5.243
- net di_13: now also U5.241
- net di_14: now also U5.251
- net di_15: now also U5.242
- net di_16: now also U5.257
- net di_17: now also U5.250
- net di_18: now also U5.262
- net di_19: now also U5.248
- net di_2: now also U5.223
- net di_20: now also U5.249
- net di_21: now also U5.256
- net di_22: now also U5.255
- net di_23: now also U5.275
- net di_24: now also U5.261
- net di_25: now also U5.268
- net di_26: now also U5.260
- net di_27: now also U5.292
- net di_28: now also U5.267
- net di_29: now also U5.266
- net di_3: now also U5.215
- net di_30: now also U5.274
- net di_31: now also U5.273
- net di_32: now also U5.291
- net di_33: now also U5.290
- net di_34: now also U5.314
- net di_35: now also U5.289
- net di_36: now also U5.320
- net di_37: now also U5.306
- net di_38: now also U5.288
- net di_39: now also U5.305
- net di_4: now also U5.224
- net di_40: now also U5.287
- net di_41: now also U5.304
- net di_42: now also U5.303
- net di_43: now also U5.286
- net di_44: now also U5.302
- net di_45: now also U5.301
- net di_46: now also U5.285
- net di_47: now also U5.319
- net di_5: now also U5.230
- net di_6: now also U5.229
- net di_7: now also U5.231
- net di_8: now also U5.225
- net di_9: now also U5.236
- net mclk_pause: now also U5.197
- net miso: now also U5.172
- net mosi: now also U5.196
- net pin_1: now also U5.160
- net pin_10: now also U5.151
- net pin_100: now also U5.61
- net pin_101: now also U5.60
- net pin_102: now also U5.59
- net pin_103: now also U5.58
- net pin_104: now also U5.57
- net pin_105: now also U5.56
- net pin_106: now also U5.55
- net pin_107: now also U5.54
- net pin_108: now also U5.53
- net pin_109: now also U5.52
- net pin_11: now also U5.150
- net pin_110: now also U5.51
- net pin_111: now also U5.50
- net pin_112: now also U5.49
- net pin_113: now also U5.48
- net pin_114: now also U5.47
- net pin_115: now also U5.46
- net pin_116: now also U5.45
- net pin_117: now also U5.44
- net pin_118: now also U5.43
- net pin_119: now also U5.42
- net pin_12: now also U5.149
- net pin_120: now also U5.41
- net pin_121: now also U5.40
- net pin_122: now also U5.39
- net pin_123: now also U5.38
- net pin_124: now also U5.37
- net pin_125: now also U5.36
- net pin_126: now also U5.35
- net pin_127: now also U5.34
- net pin_128: now also U5.33
- net pin_129: now also U5.32
- net pin_13: now also U5.148
- net pin_130: now also U5.31
- net pin_131: now also U5.30
- net pin_132: now also U5.29
- net pin_133: now also U5.28
- net pin_134: now also U5.27
- net pin_135: now also U5.26
- net pin_136: now also U5.25
- net pin_137: now also U5.24
- net pin_138: now also U5.23
- net pin_139: now also U5.22
- net pin_14: now also U5.147
- net pin_140: now also U5.21
- net pin_141: now also U5.20
- net pin_142: now also U5.19
- net pin_143: now also U5.18
- net pin_144: now also U5.17
- net pin_145: now also U5.16
- net pin_146: now also U5.15
- net pin_147: now also U5.14
- net pin_148: now also U5.13
- net pin_149: now also U5.12
- net pin_15: now also U5.146
- net pin_150: now also U5.11
- net pin_151: now also U5.10
- net pin_152: now also U5.9
- net pin_153: now also U5.8
- net pin_154: now also U5.7
- net pin_155: now also U5.6
- net pin_156: now also U5.5
- net pin_157: now also U5.4
- net pin_158: now also U5.3
- net pin_159: now also U5.2
- net pin_16: now also U5.145
- net pin_160: now also U5.1
- net pin_17: now also U5.144
- net pin_18: now also U5.143
- net pin_19: now also U5.142
- net pin_2: now also U5.159
- net pin_20: now also U5.141
- net pin_21: now also U5.140
- net pin_22: now also U5.139
- net pin_23: now also U5.138
- net pin_24: now also U5.137
- net pin_25: now also U5.136
- net pin_26: now also U5.135
- net pin_27: now also U5.134
- net pin_28: now also U5.133
- net pin_29: now also U5.132
- net pin_3: now also U5.158
- net pin_30: now also U5.131
- net pin_31: now also U5.130
- net pin_32: now also U5.129
- net pin_33: now also U5.128
- net pin_34: now also U5.127
- net pin_35: now also U5.126
- net pin_36: now also U5.125
- net pin_37: now also U5.124
- net pin_38: now also U5.123
- net pin_39: now also U5.122
- net pin_4: now also U5.157
- net pin_40: now also U5.121
- net pin_41: now also U5.120
- net pin_42: now also U5.119
- net pin_43: now also U5.118
- net pin_44: now also U5.117
- net pin_45: now also U5.116
- net pin_46: now also U5.115
- net pin_47: now also U5.114
- net pin_48: now also U5.113
- net pin_49: now also U5.112
- net pin_5: now also U5.156
- net pin_50: now also U5.111
- net pin_51: now also U5.110
- net pin_52: now also U5.109
- net pin_53: now also U5.108
- net pin_54: now also U5.107
- net pin_55: now also U5.106
- net pin_56: now also U5.105
- net pin_57: now also U5.104
- net pin_58: now also U5.103
- net pin_59: now also U5.102
- net pin_6: now also U5.155
- net pin_60: now also U5.101
- net pin_61: now also U5.100
- net pin_62: now also U5.99
- net pin_63: now also U5.98
- net pin_64: now also U5.97
- net pin_65: now also U5.96
- net pin_66: now also U5.95
- net pin_67: now also U5.94
- net pin_68: now also U5.93
- net pin_69: now also U5.92
- net pin_7: now also U5.154
- net pin_70: now also U5.91
- net pin_71: now also U5.90
- net pin_72: now also U5.89
- net pin_73: now also U5.88
- net pin_74: now also U5.87
- net pin_75: now also U5.86
- net pin_76: now also U5.85
- net pin_77: now also U5.84
- net pin_78: now also U5.83
- net pin_79: now also U5.82
- net pin_8: now also U5.153
- net pin_80: now also U5.81
- net pin_81: now also U5.80
- net pin_82: now also U5.79
- net pin_83: now also U5.78
- net pin_84: now also U5.77
- net pin_85: now also U5.76
- net pin_86: now also U5.75
- net pin_87: now also U5.74
- net pin_88: now also U5.73
- net pin_89: now also U5.72
- net pin_9: now also U5.152
- net pin_90: now also U5.71
- net pin_91: now also U5.70
- net pin_92: now also U5.69
- net pin_93: now also U5.68
- net pin_94: now also U5.67
- net pin_95: now also U5.66
- net pin_96: now also U5.65
- net pin_97: now also U5.64
- net pin_98: now also U5.63
- net pin_99: now also U5.62
- net read_dac_config_0: now also U5.307
- net read_dac_config_1: now also U5.272
- net read_dac_config_2: now also U5.276
- net read_dac_config_3: now also U5.265
- net read_dac_en: now also U5.186
- net read_ref_0: now also U5.284
- net read_ref_1: now also U5.312
- net read_ref_2: now also U5.311
- net read_ref_3: now also U5.283
- net read_ref_4: now also U5.318
- net read_ref_5: now also U5.299
- net rram_addr_0: now also U5.317
- net rram_addr_1: now also U5.310
- net rram_addr_10: now also U5.315
- net rram_addr_11: now also U5.295
- net rram_addr_12: now also U5.279
- net rram_addr_13: now also U5.294
- net rram_addr_14: now also U5.278
- net rram_addr_15: now also U5.293
- net rram_addr_2: now also U5.316
- net rram_addr_3: now also U5.282
- net rram_addr_4: now also U5.298
- net rram_addr_5: now also U5.297
- net rram_addr_6: now also U5.309
- net rram_addr_7: now also U5.281
- net rram_addr_8: now also U5.296
- net rram_addr_9: now also U5.280
- net rst_n: now also U5.214
- net sa_clk: now also U5.164
- net sa_do_0: now also U5.245
- net sa_do_1: now also U5.239
- net sa_do_10: now also U5.183
- net sa_do_11: now also U5.228
- net sa_do_12: now also U5.227
- net sa_do_13: now also U5.221
- net sa_do_14: now also U5.222
- net sa_do_15: now also U5.203
- net sa_do_16: now also U5.217
- net sa_do_17: now also U5.210
- net sa_do_18: now also U5.218
- net sa_do_19: now also U5.187
- net sa_do_2: now also U5.252
- net sa_do_20: now also U5.211
- net sa_do_21: now also U5.212
- net sa_do_22: now also U5.204
- net sa_do_23: now also U5.205
- net sa_do_24: now also U5.188
- net sa_do_25: now also U5.189
- net sa_do_26: now also U5.166
- net sa_do_27: now also U5.190
- net sa_do_28: now also U5.174
- net sa_do_29: now also U5.191
- net sa_do_3: now also U5.240
- net sa_do_30: now also U5.175
- net sa_do_31: now also U5.167
- net sa_do_32: now also U5.192
- net sa_do_33: now also U5.176
- net sa_do_34: now also U5.177
- net sa_do_35: now also U5.161
- net sa_do_36: now also U5.193
- net sa_do_37: now also U5.178
- net sa_do_38: now also U5.179
- net sa_do_39: now also U5.194
- net sa_do_4: now also U5.244
- net sa_do_40: now also U5.162
- net sa_do_41: now also U5.169
- net sa_do_42: now also U5.168
- net sa_do_43: now also U5.180
- net sa_do_44: now also U5.163
- net sa_do_45: now also U5.195
- net sa_do_46: now also U5.165
- net sa_do_47: now also U5.170
- net sa_do_5: now also U5.238
- net sa_do_6: now also U5.232
- net sa_do_7: now also U5.234
- net sa_do_8: now also U5.233
- net sa_do_9: now also U5.226
- net sa_en: now also U5.313
- net sa_rdy: now also U5.171
- net sc: now also U5.181
- net sclk: now also U5.200
- net set_rst: now also U5.300
- net sl_en: now also U5.308
- net we: now also U5.277
- net wl_dac_config_0: now also U5.271
- net wl_dac_config_1: now also U5.259
- net wl_dac_config_2: now also U5.264
- net wl_dac_config_3: now also U5.270
- net wl_dac_config_4: now also U5.258
- net wl_dac_config_5: now also U5.269
- net wl_dac_config_6: now also U5.254
- net wl_dac_config_7: now also U5.263
- net wl_dac_en: now also U5.253
- net wl_en: now also U5.246
Other:
- note added: "NOTE: Clocks are re-routed to clock-capable (CC) pins"
- note added: "Pinmap"
- note removed: "di_36 iref_test di_47 read_ref_4 rram_addr_0 rram_addr_2 rram_addr_10 di_34 sa_en read_ref_1 read_ref_2 rram_addr_1 rram_addr_6 sl_en read_dac_config_0 di_37 di_39 di_41 di_42 di_44 di_45 set_rst read_ref_5 rram_addr_4 rram_addr_5 rram_addr_8 rram_addr_11 rram_addr_13 rram_addr_15 di_27 di_32 di_33 di_35 di_38 di_40 di_43 di_46 read_ref_0 read_ref_3 rram_addr_3 rram_addr_7 rram_addr_9 rram_addr_1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"
- moved on the sheet: C1, C10, C2, C3, C4, C5, C6, C7, C8, C9, D1, FB1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
