File: ember-pcb.kicad_sch (KiCad schematic)
At the start: 33 parts, among them J1 Samtec_ASP-134602-01, J2 Conn_Coaxial_Power, J3 Conn_02x12_Odd_Even, J4 Conn_01x07, J5 Conn_Coaxial_Power, SW1 SW_SP3T, SW2 SW_SP3T, SW3 SW_DIP_x02, U1 EMBER Macro, U2 LP5912-0.9DRV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

Commit message: DRC/LVS clean
Connections:
- net pin_10 renamed read_ref_2
- net pin_100 renamed sa_do_13
- net pin_103 renamed sa_do_18
- net pin_104 renamed sa_do_16
- net pin_107 renamed rst_n
- net pin_109 renamed sa_do_21
- net pin_11 renamed rram_addr_1
- net pin_110 renamed sa_do_20
- net pin_111 renamed sa_do_17
- net pin_116 renamed sa_do_23
- net pin_117 renamed sa_do_22
- net pin_118 renamed sa_do_15
- net pin_12 renamed rram_addr_6
- net pin_121 renamed sclk
- net pin_126 renamed sa_do_45
- net pin_127 renamed sa_do_39
- net pin_128 renamed sa_do_36
- net pin_129 renamed sa_do_32
- net pin_13 renamed sl_en
- net pin_130 renamed sa_do_29
- net pin_131 renamed sa_do_27
- net pin_132 renamed sa_do_25
- net pin_133 renamed sa_do_24
- net pin_134 renamed sa_do_19
- net pin_135 renamed read_dac_en
- net pin_138 renamed sa_do_10
- net pin_14 renamed read_dac_config_0
- net pin_140 renamed sc
- net pin_141 renamed sa_do_43
- net pin_142 renamed sa_do_38
- net pin_143 renamed sa_do_37
- net pin_144 renamed sa_do_34
- net pin_145 renamed sa_do_33
- net pin_146 renamed sa_do_30
- net pin_147 renamed sa_do_28
- net pin_150 renamed sa_rdy
- net pin_151 renamed sa_do_47
- net pin_152 renamed sa_do_41
- net pin_153 renamed sa_do_42
- net pin_154 renamed sa_do_31
- net pin_155 renamed sa_do_26
- net pin_156 renamed sa_do_46
- net pin_157 renamed sa_clk
- net pin_158 renamed sa_do_44
- net pin_159 renamed sa_do_40
- net pin_160 renamed sa_do_35
- net pin_21 renamed set_rst
- net pin_22 renamed read_ref_5
- net pin_23 renamed rram_addr_4
- net pin_24 renamed rram_addr_5
- net pin_25 renamed rram_addr_8
- net pin_26 renamed rram_addr_11
- net pin_27 renamed rram_addr_13
- net pin_28 renamed rram_addr_15
- net pin_3 renamed read_ref_4
- net pin_37 renamed read_ref_0
- net pin_38 renamed read_ref_3
- net pin_39 renamed rram_addr_3
- net pin_4 renamed rram_addr_0
- net pin_40 renamed rram_addr_7
- net pin_41 renamed rram_addr_9
- net pin_42 renamed rram_addr_12
- net pin_43 renamed rram_addr_14
- net pin_44 renamed we
- net pin_45 renamed read_dac_config_2
- net pin_49 renamed read_dac_config_1
- net pin_5 renamed rram_addr_2
- net pin_50 renamed wl_dac_config_0
- net pin_51 renamed wl_dac_config_3
- net pin_52 renamed wl_dac_config_5
- net pin_56 renamed read_dac_config_3
- net pin_57 renamed wl_dac_config_2
- net pin_58 renamed wl_dac_config_7
- net pin_6 renamed rram_addr_10
- net pin_62 renamed wl_dac_config_1
- net pin_63 renamed wl_dac_config_4
- net pin_67 renamed wl_dac_config_6
- net pin_68 renamed wl_dac_en
- net pin_69 renamed sa_do_2
- net pin_75 renamed wl_en
- net pin_76 renamed sa_do_0
- net pin_77 renamed sa_do_4
- net pin_8 renamed sa_en
- net pin_81 renamed sa_do_3
- net pin_82 renamed sa_do_1
- net pin_83 renamed sa_do_5
- net pin_87 renamed sa_do_7
- net pin_88 renamed sa_do_8
- net pin_89 renamed sa_do_6
- net pin_9 renamed read_ref_1
- net pin_93 renamed sa_do_11
- net pin_94 renamed sa_do_12
- net pin_95 renamed sa_do_9
- net pin_99 renamed sa_do_14
Other:
- note removed: "NOTE: Clocks are re-routed to clock-capable (CC) pins"
- note removed: "Pinmap"
- moved on the sheet: C1, C10, C2, C3, C4, C5, C6, C7, C8, C9, D1, FB1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
