File: ember-pcb.kicad_sch (KiCad schematic)
At the start: 33 parts, among them J1 Samtec_ASP-134602-01, J2 Conn_Coaxial_Power, J3 Conn_02x12_Odd_Even, J4 Conn_01x07, J5 Conn_Coaxial_Power, SW1 SW_SP3T, SW2 SW_SP3T, SW3 SW_DIP_x02, U1 EMBER Macro, U2 LP5912-0.9DRV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

Commit message: 12 layer board final
Parts:
- added FID1, FID2, FID3: Fiducial, Fiducial:Fiducial_1mm_Mask3mm, symbol Mechanical:Fiducial
